Commit message: Basicly finish all part

File: eight-thurster/src/bluerov2/bluerov2_description/urdf/base.xacro (robot description, xacro)
@@ -88,4 +88,4 @@
     <!-- Include the sensor modules: 3D Pose, IMU, Pressure, Camera -->
     <xacro:include filename="$(find bluerov2_description)/urdf/sensors.xacro"/>
-  </xacro:macro>
+    </xacro:macro>
 </robot>

File: eight-thurster/src/bluerov2/bluerov2_description/urdf/gazebo.xacro (robot description, xacro)
@@ -40,5 +40,6 @@
           -->
           <linear_damping>
-            -11.7391 -20 -31.8678 -25 -44.9085 -5
+            <!-- -11.7391 -20 -31.8678 -25 -44.9085 -5.0000 -->
+            -4.03 -6.22 -5.18 -0.07 -0.07 -0.07
           </linear_damping>
           <!--
@@ -57,5 +58,6 @@
           -->
           <quadratic_damping>
-            0 0 0 0 0 0
+            <!-- 0 0 0 0 0 0 -->
+            -18.18 -21.66 -36.99 -1.55 -1.55 -1.55
           </quadratic_damping>
           <!--
